File: pcb/blad_bottom_plate.kicad_sch (KiCad schematic)
At the start: 3 parts

Commit message: Update PCB and plate designs
Parts:
- removed BT1: CR2032, Smidr:BAT-SMD_MY-1632-03, symbol Device:Battery_Cell
- removed TP1: +BATT, TestPoint:TestPoint_Keystone_5019_Miniature, symbol Connector:TestPoint
- removed TP2: -BATT, TestPoint:TestPoint_Keystone_5019_Miniature, symbol Connector:TestPoint
