File: pcb/blad.kicad_sch (KiCad schematic)
At the start: 114 parts, among them J1 HRO_TYPE-C-31-M-12, J2 SWD, Q1 AO3401A, SW1 1U, SW10 1U, SW11 1U, SW12 1U, SW13 1.25U, SW14 1U, SW15 1U, SW16 1U, SW17 1U, SW18 1U, SW19 1U, SW2 1U, SW20 1U, SW21 1U, SW22 1U, SW23 1.75U, SW24 1.75U, SW25 1U, SW26 1U, SW27 1U, SW28 1U, SW29 1U, SW3 1U, SW30 1U, SW31 1U, SW32 1U, SW33 1U, SW34 1.25U, SW35 1.25U, SW36 1U, SW37 1.25U, SW38 2.75U, SW39 2.25U, SW4 1U, SW40 1.25U, SW41 1U, SW42 1.25U, SW5 1U, SW6 1U, SW7 1U, SW8 1U, SW9 1U, U1 SRV05-4, U2 MS88SF21 1Y40AI-U

Commit message: Update keyboard design and renderings
Connections:
- net GND: now also S1.3 (C); no longer S1.1 (A)
Changed lines of the file:
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@@
-	)
-	(no_connect
-		(at 144.78 151.13)
 	)
 	(no_connect
@@
 		(at 48.26 163.83)
 	)
+	(no_connect
+		(at 144.78 146.05)
+	)
 	(wire
 		(pts
@@
 	(wire
 		(pts
-			(xy 147.32 146.05) (xy 147.32 154.94)
-		)
-		(stroke
-			(width 0)
-			(type default)
-		)
-	)
-	(wire
-		(pts
 			(xy 167.64 50.8) (xy 167.64 76.2)
 		)
@@
 	(wire
 		(pts
-			(xy 144.78 146.05) (xy 147.32 146.05)
-		)
-		(stroke
-			(width 0)
-			(type default)
-		)
-	)
-	(wire
-		(pts
 			(xy 66.04 22.86) (xy 66.04 25.4)
 		)
@@
 	(wire
 		(pts
+			(xy 144.78 151.13) (xy 147.32 151.13)
+		)
+		(stroke
+			(width 0)
+			(type default)
+		)
+	)
+	(wire
+		(pts
 			(xy 177.8 111.76) (xy 228.6 111.76)
 		)
@@
 		)
 		(stroke
+			(width 0)
+			(type default)
+		)
+	)
+	(wire
+		(pts
+			(xy 147.32 151.13) (xy 147.32 154.94)
+		)
+		(stroke
